Commit message: add rader and d435

File: urdf/husky_ur5_laser.xacro (robot description, xacro)
@@ -5,4 +5,5 @@
     <xacro:property name="gpu" value="$(arg gpu)" />
     <xacro:include filename="$(find ur_description)/urdf/inc/ur5_macro.xacro" />
+    <xacro:include filename="$(find husky_ur5)/urdf/laser.urdf.xacro" />
     <xacro:arg name="transmission_hw_interface" default="hardware_interface/EffortJointInterface"/>
     <xacro:ur5_robot prefix="ur5_" transmission_hw_interface="$(arg transmission_hw_interface)" />
@@ -13,11 +14,8 @@
             <origin xyz="0 0 0.25" rpy="0 0 0" />
         </joint>
-    <xacro:include filename="$(find velodyne_description)/urdf/VLP-16.urdf.xacro"/>
-    <xacro:VLP-16 parent="base_link" name="velodyne" topic="/velodyne_points" hz="10" samples="440" gpu="${gpu}">
-        <origin xyz="-0.2 0 0.25" rpy="0 0 0" />
-    </xacro:VLP-16>
-    <xacro:include filename="$(find realsense_ros_gazebo)/xacro/depthcam.xacro"/>
-    <xacro:realsense_d435 sensor_name="d435" parent_link="ur5_wrist_3_link" rate="10">
-        <origin rpy="0 0 0 " xyz="0.1 0 0"/>
-    </xacro:realsense_d435>
+        <joint name="joint_husky_laser" type="fixed">
+            <parent link="base_link"/>
+            <child link="laser_base_footprint"/>
+            <origin xyz="0 0 0.4" rpy="0 0 0" />
+        </joint>
 </robot>
