Commit message: update function

File: urdf/husky_ur5.xacro (robot description, xacro)
@@ -17,7 +17,7 @@
         <origin xyz="-0.2 0 0.25" rpy="0 0 0" />
     </xacro:VLP-16>
-    <xacro:include filename="$(find realsense_ros_gazebo)/xacro/depthcam.xacro"/>
-    <xacro:realsense_d435 sensor_name="d435" parent_link="ur5_wrist_3_link" rate="10">
-        <origin rpy="0 0 0 " xyz="0.1 0 0"/>
-    </xacro:realsense_d435>
+    <xacro:include filename="$(find realsense2_description)/urdf/_d435.urdf.xacro" />
+    <xacro:sensor_d435 name="camera" topics_ns="camera" parent="ur5_wrist_3_link" publish_pointcloud="true">
+        <origin xyz="0.1 0 0" rpy="0 -1.57 0" />
+    </xacro:sensor_d435>
 </robot>
